File: Isolate_ST-Link.kicad_pcb (KiCad board)
At the start: 2 copper layers, 39.5 x 38 mm, 66 parts, among them J1 USB_OTG, J2 CONN_01X06, J3 CONN_01X04, J4 CONN_01X02, J5 CONN_01X02, J6 GS2, Q1 BSS138, U1 MAU10x, U2 ADuM4160, U3 APE8865NR-33-HF-3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

Commit message: 微調整
Routing:
- net GND: track 275.5 -> 282.5 mm, vias 52 -> 54
Other:
- board text added: "Isolate_ST-Link"
- board text added: "NRST"
- board text added: "SWCLK"
- board text added: "SWDIO"
- board text added: "SWO"
Changed lines of the file:
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@@
     (area 153.449999 49.949999 193.050001 88.050001)
     (thickness 1.6)
-    (drawings 42)
-    (tracks 800)
+    (drawings 47)
+    (tracks 809)
     (zones 0)
     (modules 66)
@@
     (descr "JST EH series connector, S04B-EH, 2.50mm pitch, side entry")
     (tags "connector jst eh side horizontal angled")
-    (fp_text reference J3 (at -2.2 2.8 270) (layer F.SilkS)
+    (fp_text reference J3 (at -1.8 2.8 270) (layer F.SilkS)
       (effects (font (size 1 1) (thickness 0.15)))
     )
@@
     )
   )
-  (gr_text 3V3 (at 190 63.7) (layer B.SilkS)
+  (gr_text Isolate_ST-Link (at 180 72.7 90) (layer B.SilkS)
     (effects (font (size 1.5 1.5) (thickness 0.3)) (justify mirror))
   )
-  (gr_text Vtgt (at 168.9 85 90) (layer B.SilkS)
-    (effects (font (size 1.5 1.5) (thickness 0.3)) (justify mirror))
+  (gr_text SWO (at 156.3 84 90) (layer B.SilkS)
+    (effects (font (size 1.2 1.2) (thickness 0.27)) (justify mirror))
+  )
+  (gr_text NRST (at 158.8 84.4 90) (layer B.SilkS)
+    (effects (font (size 1.2 1.2) (thickness 0.27)) (justify mirror))
+  )
+  (gr_text SWDIO (at 161.3 84.9 90) (layer B.SilkS)
+    (effects (font (size 1.2 1.2) (thickness 0.27)) (justify mirror))
   )
-  (gr_text GND (at 163.9 85.2 90) (layer B.SilkS)
+  (gr_text SWCLK (at 166.3 85 90) (layer B.SilkS)
+    (effects (font (size 1.2 1.2) (thickness 0.27)) (justify mirror))
+  )
+  (gr_text 3V3 (at 190 63.7) (layer B.SilkS)
     (effects (font (size 1.5 1.5) (thickness 0.3)) (justify mirror))
   )
+  (gr_text Vtgt (at 168.8 84 90) (layer B.SilkS)
+    (effects (font (size 1.2 1.2) (thickness 0.27)) (justify mirror))
+  )
+  (gr_text GND (at 163.8 84 90) (layer B.SilkS)
+    (effects (font (size 1.2 1.2) (thickness 0.27)) (justify mirror))
+  )
   (gr_line (start 190.5 75.5) (end 190.5 76.9) (layer B.SilkS) (width 0.2))
   (gr_line (start 189.8 76.2) (end 190.5 75.5) (layer B.SilkS) (width 0.2))
@@
     (effects (font (size 1.5 1.5) (thickness 0.3)) (justify mirror))
   )
-  (gr_text SWD (at 162 78.1) (layer F.SilkS)
+  (gr_text SWD (at 162.5 79.2) (layer F.SilkS)
     (effects (font (size 1.5 1.5) (thickness 0.3)))
   )
@@
   (gr_line (start 184 85) (end 183.6 85) (layer F.SilkS) (width 0.2))
   (gr_line (start 184.1 85.1) (end 184 85) (layer F.SilkS) (width 0.2))
-  (dimension 39 (width 0.3) (layer Eco1.User)
-    (gr_text "39.000 mm" (at 196.35 69.5 270) (layer Eco1.User)
+  (dimension 38 (width 0.3) (layer Eco1.User)
+    (gr_text "38.000 mm" (at 196.35 69 270) (layer Eco1.User)
       (effects (font (size 1.5 1.5) (thickness 0.3)))
     )
-    (feature1 (pts (xy 193 89) (xy 197.7 89)))
+    (feature1 (pts (xy 193 88) (xy 197.7 88)))
     (feature2 (pts (xy 193 50) (xy 197.7 50)))
-    (crossbar (pts (xy 195 50) (xy 195 89)))
-    (arrow1a (pts (xy 195 89) (xy 194.413579 87.873496)))
-    (arrow1b (pts (xy 195 89) (xy 195.586421 87.873496)))
+    (crossbar (pts (xy 195 50) (xy 195 88)))
+    (arrow1a (pts (xy 195 88) (xy 194.413579 86.873496)))
+    (arrow1b (pts (xy 195 88) (xy 195.586421 86.873496)))
     (arrow2a (pts (xy 195 50) (xy 194.413579 51.126504)))
     (arrow2b (pts (xy 195 50) (xy 195.586421 51.126504)))
@@
   (segment (start 163.075 60.95) (end 163.735 60.29) (width 0.6) (layer F.Cu) (net 3))
   (segment (start 163.735 60.29) (end 165.325001 60.29) (width 0.6) (layer F.Cu) (net 3))
+  (segment (start 179.7 74.1) (end 179.7 74.3) (width 0.25) (layer F.Cu) (net 4))
+  (segment (start 179.7 74.3) (end 179.7 75.7) (width 0.25) (layer F.Cu) (net 4))
+  (segment (start 178.65 71.55) (end 179.7 72.6) (width 0.25) (layer F.Cu) (net 4))
+  (segment (start 177.75 71.55) (end 178.65 71.55) (width 0.25) (layer F.Cu) (net 4))
+  (segment (start 179.7 72.6) (end 179.7 74.3) (width 0.25) (layer F.Cu) (net 4))
+  (segment (start 176.6 66.6) (end 177.5 66.6) (width 0.25) (layer B.Cu) (net 4))
+  (via (at 177.5 66.6) (size 0.6) (drill 0.4) (layers F.Cu B.Cu) (net 4))
+  (segment (start 174.625001 66.64) (end 176.56 66.64) (width 0.25) (layer F.Cu) (net 4))
+  (segment (start 176.56 66.64) (end 176.6 66.6) (width 0.25) (layer F.Cu) (net 4))
+  (via (at 176.6 66.6) (size 0.6) (drill 0.4) (layers F.Cu B.Cu) (net 4))
   (segment (start 171.15 69.45) (end 171.15 70.7) (width 0.25) (layer F.Cu) (net 4))
   (segment (start 171.15 70.7) (end 171.35 70.9) (width 0.25) (layer F.Cu) (net 4))
@@
   (segment (start 181.974999 76.025001) (end 182.375001 75.624999) (width 0.25) (layer F.Cu) (net 4))
   (segment (start 182.375001 75.624999) (end 182.6 75.4) (width 0.25) (layer F.Cu) (net 4))
-  (segment (start 179.7 74.1) (end 179.7 75.7) (width 0.25) (layer F.Cu) (net 4))
   (segment (start 179.7 75.7) (end 180.1 76.1) (width 0.25) (layer F.Cu) (net 4))
   (segment (start 177.75 73.05) (end 178.65 73.05) (width 0.25) (layer F.Cu) (net 4))

Commit message: 配線の修正
Parts:
- moved R12 2.10 mm to (182.9, 78.8)
- moved R13 2.10 mm to (182.9, 76.1)
- moved C8 1.70 mm to (176.5, 81.0)
- moved D3 1.40 mm to (181.2, 79.1)
- moved D4 1.40 mm to (181.2, 75.8)
- moved D9 1.10 mm to (183.6, 52.9)
- moved D10 0.80 mm to (183.6, 60.7)
- moved D7 0.50 mm to (185.5, 85.1)
- moved D8 0.50 mm to (185.5, 86.8)
- moved R27 0.50 mm to (174.8, 85.5)
- moved R28 0.50 mm to (174.8, 87.1)
- moved R21 0.21 mm to (175.0, 79.6), turned to 0 degrees
- moved D6 0.10 mm to (186.1, 70.0)
Routing:
- net GND: track 282.5 -> 394.8 mm, vias 54 -> 109
- net +3V3: track 150.2 -> 104.1 mm, vias 4 -> 8
- net GNDPWR: track 156.0 -> 161.1 mm
- net Net-(C8-Pad1): track 4.07 -> 5.88 mm
- net /MCU/UART_TX: track 17.2 -> 18.0 mm
- net +5V: track 24.8 -> 24.1 mm
- net Net-(R27-Pad1): track 14.6 -> 15.3 mm
- net Net-(D8-Pad1): track 1.37 -> 1.87 mm
Other:
- board size 39.5 x 38 mm -> 39 x 38 mm
