File: Isolate_ST-Link.kicad_pcb (KiCad board)
At the start: 2 copper layers, 39 x 38 mm, 66 parts, among them J1 USB_OTG, J2 CONN_01X06, J3 CONN_01X04, J4 CONN_01X02, J5 CONN_01X02, J6 GS2, Q1 BSS138, U1 MAU10x, U2 ADuM4160, U3 APE8865NR-33-HF-3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

Commit message: ダンピング抵抗追加 分圧抵抗に変更
Other:
- board text added: "Designed"
- board text added: "by @yuqlid"
Changed lines of the file:
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@@
     (area 153.449999 49.949999 192.550001 88.050001)
     (thickness 1.6)
-    (drawings 47)
+    (drawings 49)
     (tracks 961)
     (zones 0)
@@
     )
   )
-  (gr_text Isolate_ST-Link (at 180 72.7 90) (layer B.SilkS)
+  (gr_text "by @yuqlid" (at 165.9 62.8 90) (layer B.SilkS)
+    (effects (font (size 1.2 1.2) (thickness 0.2)) (justify mirror))
+  )
+  (gr_text Designed (at 164.2 61.1 90) (layer B.SilkS)
+    (effects (font (size 1.2 1.2) (thickness 0.2)) (justify mirror))
+  )
+  (gr_text Isolate_ST-Link (at 161.8 64.9 90) (layer B.SilkS)
     (effects (font (size 1.5 1.5) (thickness 0.3)) (justify mirror))
   )

Commit message: 部品割当して基板の修正
Parts:
- removed D11: D, Diodes_SMD:D_SOD-323
- R28: value 100 -> 22
- R29: value 10k -> 4.7k
- moved R28 10.9 mm to (167.1, 79.4)
- moved R29 3.28 mm to (174.8, 87.0)
Connections:
- J2 pad 2: T_JTCK -> Net-(J2-Pad2)
- R28 pad 1: Net-(D11-Pad1) -> Net-(J2-Pad2)
- R28 pad 2: Net-(R27-Pad1) -> T_JTCK
- R29 pad 2: GND -> Net-(R27-Pad1)
Routing:
- net GND: track 394.8 -> 389.6 mm, vias 109 -> 108
- net T_JTCK: track 21.3 -> 19.1 mm
- net Net-(J2-Pad2): track 0.00 -> 1.82 mm
- net /MCU/Vtarget: track 8.67 -> 10.2 mm
- net Net-(D11-Pad1): track 1.32 -> 0.00 mm

Commit message: 配線の修正
Parts:
- moved R27 2.05 mm to (176.2, 87.0), turned to 0 degrees
- moved R29 1.40 mm to (173.4, 87.0)
Routing:
- net GND: track 389.6 -> 387.7 mm
- net /MCU/Vtarget: track 10.2 -> 8.77 mm
- net Net-(R27-Pad1): track 15.2 -> 16.3 mm

Commit message: 修正
Routing:
- net GND: track 387.7 -> 390.0 mm, vias 108 -> 109
Changed lines of the file:
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@@
     (thickness 1.6)
     (drawings 49)
-    (tracks 958)
+    (tracks 962)
     (zones 0)
     (modules 65)
@@
   (segment (start 163.075 60.95) (end 163.735 60.29) (width 0.6) (layer F.Cu) (net 3))
   (segment (start 163.735 60.29) (end 165.325001 60.29) (width 0.6) (layer F.Cu) (net 3))
+  (segment (start 164.724999 80.275001) (end 165 80) (width 0.4) (layer B.Cu) (net 4))
+  (segment (start 165 80) (end 165 79.4) (width 0.4) (layer B.Cu) (net 4))
+  (via (at 165 79.4) (size 0.8) (drill 0.6) (layers F.Cu B.Cu) (net 4))
+  (segment (start 163.8 81.2) (end 164.724999 80.275001) (width 0.4) (layer B.Cu) (net 4))
   (segment (start 172.7 85) (end 172.7 85.4) (width 0.25) (layer F.Cu) (net 4))
   (segment (start 177.8 85.4) (end 172.7 85.4) (width 0.25) (layer F.Cu) (net 4))

Commit message: 進捗
Parts:
- added R30: 0, Resistors_SMD:R_0603, F.Cu at (179.0, 91.1)
- added R31: 0, Resistors_SMD:R_0603, F.Cu at (172.4, 91.5)
- added R32: 0, Resistors_SMD:R_0603, F.Cu at (166.0, 92.1)
- added R33: 0, Resistors_SMD:R_0603, F.Cu at (168.8, 96.3)
- added R34: 10k, Resistors_SMD:R_0603, F.Cu at (173.0, 98.1)
Connections:
- net Net-(C8-Pad1) renamed SYS_NRST
- R28 pad 1: Net-(J2-Pad2) -> T_JTCK
- R28 pad 2: T_JTCK -> Net-(J2-Pad2)
- U4 pad 34: Net-(U4-Pad34) -> SYS_JTMS
- U4 pad 37: Net-(U4-Pad37) -> SYS_JTCK
Routing:
- net T_JTCK: track 19.1 -> 9.00 mm
- net Net-(J2-Pad2): track 1.82 -> 11.9 mm

Commit message: 進捗
Parts:
- R34: moved to B.Cu
- moved R34 23.3 mm to (170.6, 74.8), turned to 180 degrees
- moved R33 20.7 mm to (166.2, 75.8), turned to 270 degrees
- moved R30 19.0 mm to (167.8, 75.8), turned to 270 degrees
- moved R31 18.2 mm to (163.2, 75.8), turned to 270 degrees
- moved R32 16.4 mm to (164.8, 75.8), turned to 270 degrees
- moved C11 1.50 mm to (175.8, 73.5)
- moved C8 1.50 mm to (178.0, 81.0)
- moved J6 1.50 mm to (170.7, 72.7)
- moved R21 1.50 mm to (176.5, 79.6)
- moved R22 1.50 mm to (177.6, 70.0)
- moved R23 1.50 mm to (173.3, 79.0)
- moved R24 1.50 mm to (172.7, 73.7)
- moved R25 1.50 mm to (172.6, 81.0)
- moved R26 1.50 mm to (175.6, 71.5)
- moved U4 1.50 mm to (174.9, 73.8)
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Connections:
- R31 pad 2: T_NRST -> Net-(J2-Pad5)
- R32 pad 2: T_JTMS -> Net-(J2-Pad4)
- R33 pad 2: T_JTCK -> Net-(J2-Pad2)
Routing:
- net GND: track 390.0 -> 329.0 mm, vias 109 -> 85
- net SYS_NRST: track 5.88 -> 20.7 mm
- net SYS_JTMS: track 0.00 -> 13.0 mm, vias 0 -> 2
- net T_JTCK: track 9.00 -> 20.8 mm
- net Net-(J2-Pad5): track 1.82 -> 9.01 mm
- net SYS_JTCK: track 0.00 -> 6.26 mm
- net Net-(J2-Pad4): track 1.82 -> 7.95 mm
- net Net-(J2-Pad2): track 11.9 -> 6.54 mm
- net /MCU/Vtarget: track 8.77 -> 13.9 mm
- net +3V3: track 104.1 -> 100.3 mm, vias 8 -> 10
- net /MCU/USB_RENUMn: track 17.2 -> 13.8 mm
- net Net-(J6-Pad1): track 3.09 -> 5.39 mm
- net /MCU/LED_STLINK: track 19.2 -> 20.9 mm
- net T_SWO: track 23.4 -> 25.0 mm
- net T_JTMS: track 23.3 -> 24.8 mm
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
Commit message: AW修正
Parts:
- moved R27 3.50 mm to (179.7, 87.0)
- moved R29 3.40 mm to (176.8, 87.0)
- moved R30 1.65 mm to (166.1, 75.7)
- moved R31 1.65 mm to (161.6, 75.7)
- moved R32 1.65 mm to (163.1, 75.7)
- moved R33 1.65 mm to (164.6, 75.7)
- moved C8 1.30 mm to (176.7, 81.0)
- moved R23 1.20 mm to (172.4, 79.8), turned to 180 degrees
- moved R25 0.38 mm to (172.4, 81.3)
- moved R24 0.35 mm to (172.7, 73.3)
- moved R21 0.30 mm to (176.2, 79.6), turned to 180 degrees
- turned R34 to 0 degrees
Routing:
- net +3V3: track 100.3 -> 137.5 mm, vias 10 -> 9
- net GND: track 329.0 -> 318.4 mm, vias 85 -> 83
- net /MCU/Vtarget: track 13.9 -> 18.6 mm
- net Net-(R27-Pad1): track 15.0 -> 12.1 mm
- net SYS_JTMS: track 13.0 -> 14.3 mm
- net SYS_JTCK: track 6.26 -> 7.57 mm
- net Net-(J2-Pad5): track 9.01 -> 8.18 mm
- net Net-(J2-Pad2): track 6.54 -> 7.35 mm
- net Net-(J2-Pad4): track 7.95 -> 7.32 mm
- net SYS_NRST: track 20.7 -> 20.1 mm
Other:
- board text removed: "Vtgt"

Commit message: 進捗
Parts:
- moved R21 0.80 mm to (176.2, 78.8)
- moved R7 0.70 mm to (180.1, 64.7)
- moved R26 0.64 mm to (175.9, 72.0)
- moved C11 0.50 mm to (175.8, 74.0)
- moved C8 0.25 mm to (176.7, 80.8)
- moved R30 0.20 mm to (166.1, 75.5)
- moved R31 0.20 mm to (161.6, 75.5)
- moved R32 0.20 mm to (163.1, 75.5)
- moved R33 0.20 mm to (164.6, 75.5)
Routing:
- net GND: track 318.4 -> 336.2 mm, vias 83 -> 93
- net SYS_NRST: track 20.1 -> 21.1 mm
- net T_JTMS: track 24.8 -> 23.9 mm
- net +3V3: track 137.5 -> 138.4 mm
- net /MCU/LED_STLINK: track 20.9 -> 21.5 mm
