File: Isolate_ST-Link.sch (KiCad schematic (older format))
At the start: 50 parts, among them J1 USB_OTG, J2 CONN_01X06, J3 CONN_01X04, J4 CONN_01X02, J5 CONN_01X02, Q1 BSS138, U1 MAU10x, U2 ADuM4160, U3 APE8865NR-33-HF-3

Commit message: https://github.com/Yuqlid/Isolate_ST-Link/projects/1#card-5148549 プルダウン抵抗追加
Connections:
- wire segments 90 -> 91
Changed lines of the file:
@@
 L R R14
 U 1 1 5948BD9F
-P 8350 3500
-F 0 "R14" V 8430 3500 50  0000 C CNN
-F 1 "22" V 8350 3500 50  0000 C CNN
-F 2 "Resistors_SMD:R_0603" V 8280 3500 50  0001 C CNN
-F 3 "" H 8350 3500 50  0001 C CNN
-	1    8350 3500
+P 8150 3500
+F 0 "R14" V 8230 3500 50  0000 C CNN
+F 1 "22" V 8150 3500 50  0000 C CNN
+F 2 "Resistors_SMD:R_0603" V 8080 3500 50  0001 C CNN
+F 3 "" H 8150 3500 50  0001 C CNN
+	1    8150 3500
 	0    1    1    0
 $EndComp
@@
 	8500 3200 7450 3200
 Wire Wire Line
-	7950 3500 8200 3500
+	7950 3500 8000 3500
 Wire Wire Line
 	8200 3600 7950 3600
@@
 L R R28
 U 1 1 59CA9CFA
-P 8300 3300
-F 0 "R28" V 8380 3300 50  0000 C CNN
-F 1 "22" V 8300 3300 50  0000 C CNN
-F 2 "Resistors_SMD:R_0603" V 8230 3300 50  0001 C CNN
-F 3 "" H 8300 3300 50  0001 C CNN
-	1    8300 3300
+P 8150 3300
+F 0 "R28" V 8230 3300 50  0000 C CNN
+F 1 "22" V 8150 3300 50  0000 C CNN
+F 2 "Resistors_SMD:R_0603" V 8080 3300 50  0001 C CNN
+F 3 "" H 8150 3300 50  0001 C CNN
+	1    8150 3300
 	0    1    1    0
 $EndComp
 Wire Wire Line
-	8450 3300 8500 3300
-Wire Wire Line
-	8150 3300 7950 3300
+	8300 3300 8500 3300
+Wire Wire Line
+	8000 3300 7950 3300
+Wire Wire Line
+	8250 3500 8500 3500
 $EndSCHEMATC

Commit message: 修正
Connections:
- wire segments 91 -> 89

Commit message: 書き込みようの抵抗を追加
Parts:
- added R? (x4): 0, Resistors_SMD:R_0603, symbol R
Connections:
- net labels added: SYS_JTCK, SYS_JTMS, SYS_NRST
- wire segments 89 -> 99
Changed lines of the file:
@@
 L CONN_01X06 J2
 U 1 1 5948A2BD
-P 8700 2950
-F 0 "J2" H 8700 3300 50  0000 C CNN
-F 1 "CONN_01X06" V 8800 2950 50  0000 C CNN
-F 2 "Connectors_JST:JST_EH_S06B-EH_06x2.50mm_Angled" H 8700 2950 50  0001 C CNN
-F 3 "" H 8700 2950 50  0001 C CNN
-	1    8700 2950
+P 10300 2950
+F 0 "J2" H 10300 3300 50  0000 C CNN
+F 1 "CONN_01X06" V 10400 2950 50  0000 C CNN
+F 2 "Connectors_JST:JST_EH_S06B-EH_06x2.50mm_Angled" H 10300 2950 50  0001 C CNN
+F 3 "" H 10300 2950 50  0001 C CNN
+	1    10300 2950
 	1    0    0    1
 $EndComp
-Text GLabel 7950 2700 0    60   Input ~ 0
+Text GLabel 9150 2700 0    60   Input ~ 0
 T_SWO
-Text GLabel 7550 2800 0    60   Input ~ 0
+Text GLabel 9150 2800 0    60   Input ~ 0
 T_NRST
-Text GLabel 7950 2900 0    60   Input ~ 0
+Text GLabel 9150 2900 0    60   Input ~ 0
 T_JTMS
 $Comp
 L GND #PWR08
 U 1 1 5948BBA0
-P 8150 3000
-F 0 "#PWR08" H 8150 2750 50  0001 C CNN
-F 1 "GND" H 8150 2850 50  0000 C CNN
-F 2 "" H 8150 3000 50  0001 C CNN
-F 3 "" H 8150 3000 50  0001 C CNN
-	1    8150 3000
+P 9200 3000
+F 0 "#PWR08" H 9200 2750 50  0001 C CNN
+F 1 "GND" H 9200 2850 50  0000 C CNN
+F 2 "" H 9200 3000 50  0001 C CNN
+F 3 "" H 9200 3000 50  0001 C CNN
+	1    9200 3000
 	0    1    -1   0
 $EndComp
-Text GLabel 7950 3100 0    60   Input ~ 0
+Text GLabel 9150 3100 0    60   Input ~ 0
 T_JTCK
 $Comp
 L R R14
 U 1 1 5948BD9F
-P 8300 2900
-F 0 "R14" V 8380 2900 50  0000 C CNN
-F 1 "22" V 8300 2900 50  0000 C CNN
-F 2 "Resistors_SMD:R_0603" V 8230 2900 50  0001 C CNN
-F 3 "" H 8300 2900 50  0001 C CNN
-	1    8300 2900
+P 9900 2900
+F 0 "R14" V 9980 2900 50  0000 C CNN
+F 1 "22" V 9900 2900 50  0000 C CNN
+F 2 "Resistors_SMD:R_0603" V 9830 2900 50  0001 C CNN
+F 3 "" H 9900 2900 50  0001 C CNN
+	1    9900 2900
 	0    1    -1   0
 $EndComp
@@
 L R R15
 U 1 1 59498AC7
-P 8100 2800
-F 0 "R15" V 8180 2800 50  0000 C CNN
-F 1 "22" V 8100 2800 50  0000 C CNN
-F 2 "Resistors_SMD:R_0603" V 8030 2800 50  0001 C CNN
-F 3 "" H 8100 2800 50  0001 C CNN
-	1    8100 2800
+P 9700 2800
+F 0 "R15" V 9780 2800 50  0000 C CNN
+F 1 "22" V 9700 2800 50  0000 C CNN
+F 2 "Resistors_SMD:R_0603" V 9630 2800 50  0001 C CNN
+F 3 "" H 9700 2800 50  0001 C CNN
+	1    9700 2800
 	0    1    -1   0
 $EndComp
@@
 L R R16
 U 1 1 59498B28
-P 8300 2700
-F 0 "R16" V 8380 2700 50  0000 C CNN
-F 1 "22" V 8300 2700 50  0000 C CNN
-F 2 "Resistors_SMD:R_0603" V 8230 2700 50  0001 C CNN
-F 3 "" H 8300 2700 50  0001 C CNN
-	1    8300 2700
+P 9900 2700
+F 0 "R16" V 9980 2700 50  0000 C CNN
+F 1 "22" V 9900 2700 50  0000 C CNN
+F 2 "Resistors_SMD:R_0603" V 9830 2700 50  0001 C CNN
+F 3 "" H 9900 2700 50  0001 C CNN
+	1    9900 2700
 	0    1    -1   0
 $EndComp
@@
 L R R28
 U 1 1 59CA9CFA
-P 8300 3100
-F 0 "R28" V 8380 3100 50  0000 C CNN
-F 1 "22" V 8300 3100 50  0000 C CNN
-F 2 "Resistors_SMD:R_0603" V 8230 3100 50  0001 C CNN
-F 3 "" H 8300 3100 50  0001 C CNN
-	1    8300 3100
+P 9900 3100
+F 0 "R28" V 9980 3100 50  0000 C CNN
+F 1 "22" V 9900 3100 50  0000 C CNN
+F 2 "Resistors_SMD:R_0603" V 9830 3100 50  0001 C CNN
+F 3 "" H 9900 3100 50  0001 C CNN
+	1    9900 3100
+	0    -1   1    0
+$EndComp
+Text GLabel 8800 2350 0    60   Input ~ 0
+SYS_JTMS
+Text GLabel 8800 2500 0    60   Input ~ 0
+SYS_JTCK
+$Comp
+L R R?
+U 1 1 59E58B29
+P 9000 2350
+F 0 "R?" V 9080 2350 50  0000 C CNN
+F 1 "0" V 9000 2350 50  0000 C CNN
+F 2 "Resistors_SMD:R_0603" V 8930 2350 50  0001 C CNN
+F 3 "" H 9000 2350 50  0001 C CNN
+	1    9000 2350
+	0    -1   1    0
+$EndComp
+$Comp
+L R R?
+U 1 1 59E595A8
+P 9000 2500
+F 0 "R?" V 9080 2500 50  0000 C CNN
+F 1 "0" V 9000 2500 50  0000 C CNN
+F 2 "Resistors_SMD:R_0603" V 8930 2500 50  0001 C CNN
+F 3 "" H 9000 2500 50  0001 C CNN
+	1    9000 2500
+	0    -1   1    0
+$EndComp
+Text GLabel 8800 2200 0    60   Input ~ 0
+SYS_NRST
+$Comp
+L R R?
+U 1 1 59E5FA0B
+P 9000 2200
+F 0 "R?" V 9080 2200 50  0000 C CNN
+F 1 "0" V 9000 2200 50  0000 C CNN
+F 2 "Resistors_SMD:R_0603" V 8930 2200 50  0001 C CNN
+F 3 "" H 9000 2200 50  0001 C CNN
+	1    9000 2200
 	0    -1   1    0
 $EndComp
@@
 Connection ~ 800  4700
 Wire Wire Line
-	8150 3000 8500 3000
+	9200 3000 10100 3000
 Wire Wire Line
 	5750 2800 5800 2800
@@
 Connection ~ 5800 2800
 Wire Wire Line
-	8500 3200 7000 3200
-Wire Wire Line
-	7950 2900 8150 2900
-Wire Wire Line
-	7950 2800 7550 2800
-Wire Wire Line
-	7950 2700 8150 2700
+	7000 3200 10100 3200
+Wire Wire Line
+	9150 2900 9750 2900
+Wire Wire Line
+	9550 2800 9150 2800
+Wire Wire Line
+	9150 2700 9750 2700
 Wire Wire Line
 	4250 3750 4250 4400
@@
 Connection ~ 1150 4050
 Wire Wire Line
-	8450 3100 8500 3100
-Wire Wire Line
-	8150 3100 7950 3100
-Wire Wire Line
-	8450 2900 8500 2900
-Wire Wire Line
-	8450 2700 8500 2700
-Wire Wire Line
-	8250 2800 8500 2800
+	10050 3100 10100 3100
+Wire Wire Line
+	9750 3100 9150 3100
+Wire Wire Line
+	10050 2900 10100 2900
+Wire Wire Line
+	10050 2700 10100 2700
+Wire Wire Line
+	9850 2800 10100 2800
+Wire Wire Line
+	8800 2350 8850 2350
+Wire Wire Line
+	8800 2500 8850 2500
+Wire Wire Line
+	8800 2200 8850 2200
+Wire Wire Line
+	9150 2500 9250 2500
+Wire Wire Line
+	9250 2500 9250 3100
+Connection ~ 9250 3100
+Wire Wire Line
+	9150 2350 9350 2350
+Wire Wire Line
+	9350 2350 9350 2900
+Connection ~ 9350 2900
+Wire Wire Line
+	9150 2200 9450 2200
+Wire Wire Line
+	9450 2200 9450 2800
+Connection ~ 9450 2800
+$Comp
+L R R?
+U 1 1 59E61735
+P 8200 3000
+F 0 "R?" V 8280 3000 50  0000 C CNN
+F 1 "0" V 8200 3000 50  0000 C CNN
+F 2 "Resistors_SMD:R_0603" V 8130 3000 50  0001 C CNN
+F 3 "" H 8200 3000 50  0001 C CNN
+	1    8200 3000
+	-1   0    0    -1
+$EndComp
+$Comp
+L +3V3 #PWR?
+U 1 1 59E61D26
+P 8200 2850
+F 0 "#PWR?" H 8200 2700 50  0001 C CNN
+F 1 "+3V3" H 8200 2990 50  0000 C CNN
+F 2 "" H 8200 2850 50  0001 C CNN
+F 3 "" H 8200 2850 50  0001 C CNN
+	1    8200 2850
+	1    0    0    -1
+$EndComp
+Wire Wire Line
+	8200 3150 8200 3200
+Connection ~ 8200 3200
 $EndSCHEMATC

Commit message: 進捗
Parts:
- gave numbers to parts that had none: 4
Changed lines of the file:
@@
 SYS_JTCK
 $Comp
-L R R?
+L R R32
 U 1 1 59E58B29
 P 9000 2350
-F 0 "R?" V 9080 2350 50  0000 C CNN
+F 0 "R32" V 9080 2350 50  0000 C CNN
 F 1 "0" V 9000 2350 50  0000 C CNN
 F 2 "Resistors_SMD:R_0603" V 8930 2350 50  0001 C CNN
@@
 $EndComp
 $Comp
-L R R?
+L R R33
 U 1 1 59E595A8
 P 9000 2500
-F 0 "R?" V 9080 2500 50  0000 C CNN
+F 0 "R33" V 9080 2500 50  0000 C CNN
 F 1 "0" V 9000 2500 50  0000 C CNN
 F 2 "Resistors_SMD:R_0603" V 8930 2500 50  0001 C CNN
@@
 SYS_NRST
 $Comp
-L R R?
+L R R31
 U 1 1 59E5FA0B
 P 9000 2200
-F 0 "R?" V 9080 2200 50  0000 C CNN
+F 0 "R31" V 9080 2200 50  0000 C CNN
 F 1 "0" V 9000 2200 50  0000 C CNN
 F 2 "Resistors_SMD:R_0603" V 8930 2200 50  0001 C CNN
@@
 Connection ~ 9450 2800
 $Comp
-L R R?
+L R R30
 U 1 1 59E61735
 P 8200 3000
-F 0 "R?" V 8280 3000 50  0000 C CNN
+F 0 "R30" V 8280 3000 50  0000 C CNN
 F 1 "0" V 8200 3000 50  0000 C CNN
 F 2 "Resistors_SMD:R_0603" V 8130 3000 50  0001 C CNN
@@
 $EndComp
 $Comp
-L +3V3 #PWR?
+L +3V3 #PWR042
 U 1 1 59E61D26
 P 8200 2850
-F 0 "#PWR?" H 8200 2700 50  0001 C CNN
+F 0 "#PWR042" H 8200 2700 50  0001 C CNN
 F 1 "+3V3" H 8200 2990 50  0000 C CNN
 F 2 "" H 8200 2850 50  0001 C CNN

Commit message: 進捗
Changed lines of the file:
@@
 EESchema Schematic File Version 2
-LIBS:Isolate_ST-Link-rescue
 LIBS:power
 LIBS:device
@@
 LIBS:zetex
 LIBS:Zilog
-LIBS:mylib
 LIBS:Isolate_ST-Link-cache
 EELAYER 25 0
@@
 	1    0    0    1
 $EndComp
-Text GLabel 9150 2700 0    60   Input ~ 0
+Text GLabel 9200 2700 0    60   Input ~ 0
 T_SWO
-Text GLabel 9150 2800 0    60   Input ~ 0
+Text GLabel 9200 2800 0    60   Input ~ 0
 T_NRST
-Text GLabel 9150 2900 0    60   Input ~ 0
+Text GLabel 9200 2900 0    60   Input ~ 0
 T_JTMS
 $Comp
 L GND #PWR08
 U 1 1 5948BBA0
-P 9200 3000
-F 0 "#PWR08" H 9200 2750 50  0001 C CNN
-F 1 "GND" H 9200 2850 50  0000 C CNN
-F 2 "" H 9200 3000 50  0001 C CNN
-F 3 "" H 9200 3000 50  0001 C CNN
-	1    9200 3000
+P 9500 3000
+F 0 "#PWR08" H 9500 2750 50  0001 C CNN
+F 1 "GND" H 9500 2850 50  0000 C CNN
+F 2 "" H 9500 3000 50  0001 C CNN
+F 3 "" H 9500 3000 50  0001 C CNN
+	1    9500 3000
 	0    1    -1   0
 $EndComp
-Text GLabel 9150 3100 0    60   Input ~ 0
+Text GLabel 9200 3100 0    60   Input ~ 0
 T_JTCK
 $Comp
 L R R14
 U 1 1 5948BD9F
-P 9900 2900
-F 0 "R14" V 9980 2900 50  0000 C CNN
-F 1 "22" V 9900 2900 50  0000 C CNN
-F 2 "Resistors_SMD:R_0603" V 9830 2900 50  0001 C CNN
-F 3 "" H 9900 2900 50  0001 C CNN
-	1    9900 2900
+P 9650 2900
+F 0 "R14" V 9730 2900 50  0000 C CNN
+F 1 "22" V 9650 2900 50  0000 C CNN
+F 2 "Resistors_SMD:R_0603" V 9580 2900 50  0001 C CNN
+F 3 "" H 9650 2900 50  0001 C CNN
+	1    9650 2900
 	0    1    -1   0
 $EndComp
@@
 L R R15
 U 1 1 59498AC7
-P 9700 2800
-F 0 "R15" V 9780 2800 50  0000 C CNN
-F 1 "22" V 9700 2800 50  0000 C CNN
-F 2 "Resistors_SMD:R_0603" V 9630 2800 50  0001 C CNN
-F 3 "" H 9700 2800 50  0001 C CNN
-	1    9700 2800
+P 9400 2800
+F 0 "R15" V 9480 2800 50  0000 C CNN
+F 1 "22" V 9400 2800 50  0000 C CNN
+F 2 "Resistors_SMD:R_0603" V 9330 2800 50  0001 C CNN
+F 3 "" H 9400 2800 50  0001 C CNN
+	1    9400 2800
 	0    1    -1   0
 $EndComp
@@
 L R R16
 U 1 1 59498B28
-P 9900 2700
-F 0 "R16" V 9980 2700 50  0000 C CNN
-F 1 "22" V 9900 2700 50  0000 C CNN
-F 2 "Resistors_SMD:R_0603" V 9830 2700 50  0001 C CNN
-F 3 "" H 9900 2700 50  0001 C CNN
-	1    9900 2700
+P 9650 2700
+F 0 "R16" V 9730 2700 50  0000 C CNN
+F 1 "22" V 9650 2700 50  0000 C CNN
+F 2 "Resistors_SMD:R_0603" V 9580 2700 50  0001 C CNN
+F 3 "" H 9650 2700 50  0001 C CNN
+	1    9650 2700
 	0    1    -1   0
 $EndComp
@@
 L R R28
 U 1 1 59CA9CFA
-P 9900 3100
-F 0 "R28" V 9980 3100 50  0000 C CNN
-F 1 "22" V 9900 3100 50  0000 C CNN
-F 2 "Resistors_SMD:R_0603" V 9830 3100 50  0001 C CNN
-F 3 "" H 9900 3100 50  0001 C CNN
-	1    9900 3100
+P 9650 3100
+F 0 "R28" V 9730 3100 50  0000 C CNN
+F 1 "22" V 9650 3100 50  0000 C CNN
+F 2 "Resistors_SMD:R_0603" V 9580 3100 50  0001 C CNN
+F 3 "" H 9650 3100 50  0001 C CNN
+	1    9650 3100
 	0    -1   1    0
 $EndComp
@@
 Connection ~ 800  4700
 Wire Wire Line
-	9200 3000 10100 3000
+	9500 3000 10100 3000
 Wire Wire Line
 	5750 2800 5800 2800
@@
 	7000 3200 10100 3200
 Wire Wire Line
-	9150 2900 9750 2900
-Wire Wire Line
-	9550 2800 9150 2800
-Wire Wire Line
-	9150 2700 9750 2700
+	9200 2900 9500 2900
+Wire Wire Line
+	9200 2800 9250 2800
+Wire Wire Line
+	9200 2700 9500 2700
 Wire Wire Line
 	4250 3750 4250 4400
@@
 Connection ~ 1150 4050
 Wire Wire Line
-	10050 3100 10100 3100
-Wire Wire Line
-	9750 3100 9150 3100
-Wire Wire Line
-	10050 2900 10100 2900
-Wire Wire Line
-	10050 2700 10100 2700
-Wire Wire Line
-	9850 2800 10100 2800
+	9800 3100 10100 3100
+Wire Wire Line
+	9200 3100 9500 3100
+Wire Wire Line
+	9800 2900 10100 2900
+Wire Wire Line
+	9550 2800 10100 2800
 Wire Wire Line
 	8800 2350 8850 2350
@@
 	8800 2200 8850 2200
 Wire Wire Line
-	9150 2500 9250 2500
-Wire Wire Line
-	9250 2500 9250 3100
-Connection ~ 9250 3100
-Wire Wire Line
-	9150 2350 9350 2350
-Wire Wire Line
-	9350 2350 9350 2900
-Connection ~ 9350 2900
-Wire Wire Line
-	9150 2200 9450 2200
-Wire Wire Line
-	9450 2200 9450 2800
-Connection ~ 9450 2800
+	9150 2500 9850 2500
+Wire Wire Line
+	9150 2350 9950 2350
+Wire Wire Line
+	9150 2200 10050 2200
 $Comp
 L R R30
 U 1 1 59E61735
-P 8200 3000
-F 0 "R30" V 8280 3000 50  0000 C CNN
-F 1 "0" V 8200 3000 50  0000 C CNN
-F 2 "Resistors_SMD:R_0603" V 8130 3000 50  0001 C CNN
-F 3 "" H 8200 3000 50  0001 C CNN
-	1    8200 3000
+P 7300 2900
+F 0 "R30" V 7380 2900 50  0000 C CNN
+F 1 "0" V 7300 2900 50  0000 C CNN
+F 2 "Resistors_SMD:R_0603" V 7230 2900 50  0001 C CNN
+F 3 "" H 7300 2900 50  0001 C CNN
+	1    7300 2900
 	-1   0    0    -1
 $EndComp
@@
 L +3V3 #PWR042
 U 1 1 59E61D26
-P 8200 2850
-F 0 "#PWR042" H 8200 2700 50  0001 C CNN
-F 1 "+3V3" H 8200 2990 50  0000 C CNN
-F 2 "" H 8200 2850 50  0001 C CNN
-F 3 "" H 8200 2850 50  0001 C CNN
-	1    8200 2850
-	1    0    0    -1
-$EndComp
-Wire Wire Line
-	8200 3150 8200 3200
-Connection ~ 8200 3200
+P 7300 2750
+F 0 "#PWR042" H 7300 2600 50  0001 C CNN
+F 1 "+3V3" H 7300 2890 50  0000 C CNN
+F 2 "" H 7300 2750 50  0001 C CNN
+F 3 "" H 7300 2750 50  0001 C CNN
+	1    7300 2750
+	1    0    0    -1
+$EndComp
+Wire Wire Line
+	7300 3050 7300 3200
+Connection ~ 7300 3200
+Wire Wire Line
+	9800 2700 10100 2700
+Wire Wire Line
+	10050 2200 10050 2800
+Connection ~ 10050 2800
+Wire Wire Line
+	9950 2350 9950 2900
+Connection ~ 9950 2900
+Wire Wire Line
+	9850 2500 9850 3100
+Connection ~ 9850 3100
 $EndSCHEMATC

Commit message: 見た目を整理
Parts:
- C1: value 47u -> 10u
Connections:
- wire segments 99 -> 127
